File: PCB/THG_v2/THG_v2.kicad_pcb (KiCad board)
At the start: 2 copper layers, 9 parts, among them J1 Conn_01x04_Male, J2 Conn_01x04_Male, J3 Conn_01x04_Male, J4 Conn_01x06_Male, J5 Screw_Terminal_01x02, U1 mini_esp32

Commit message: adding previous gerber file
Parts:
- added R3: n/a, Resistor_THT:R_Axial_DIN0207_L6.3mm_D2.5mm_P10.16mm_Horizontal, F.Cu at (45.1, 88.1)
- J1: value Conn_01x04_Male -> AM2315_Conn
Connections:
- U1 pad 1: unconnected-(U1-Pad1) -> GND
- U1 pad 22: unconnected-(U1-Pad22) -> GND
- U1 pad 33: unconnected-(U1-Pad33) -> GND

Commit message: adding pcb pic
Parts:
- added S1: DTS-6, Lib_Kicad:DTS-6, F.Cu at (162.7, 107.0)
- J2: value Conn_01x04_Male -> LCD_conn
- J3: value Conn_01x04_Male -> RTC_Conn
- J4: value Conn_01x06_Male -> SD_card_conn
- J5: value Screw_Terminal_01x02 -> AC_in_terminal
- moved PS1 123.5 mm to (152.0, 116.4), turned to 180 degrees
- moved J4 118.9 mm to (164.3, 82.5), turned to -90 degrees
- moved J5 98.6 mm to (161.4, 121.3), turned to 90 degrees
- moved R3 94.0 mm to (139.1, 88.7)
- moved J1 84.6 mm to (164.3, 67.2), turned to -90 degrees
- moved J3 63.9 mm to (123.2, 96.9), turned to 90 degrees
- moved R2 63.7 mm to (139.1, 78.6)
- moved R1 63.5 mm to (139.1, 83.6)
- moved J2 50.3 mm to (123.2, 82.1), turned to 90 degrees
- moved U1 10.5 mm to (143.9, 82.1)
Connections:
- J1 pad 3: Net-(J1-Pad3) -> SDA
- J1 pad 4: Net-(J1-Pad4) -> SCL
- R1 pad 1: Net-(J1-Pad3) -> +5V
- R2 pad 1: Net-(J1-Pad4) -> +5V
- R3 pad 2: unconnected-(R3-Pad2) -> Net-(S1-Pad1)
Routing:
- net +5V: track 0.00 -> 171.6 mm
- net GND: track 0.00 -> 156.2 mm
- net SDA: track 0.00 -> 74.8 mm
- net SCL: track 0.00 -> 60.7 mm
- net Net-(S1-Pad1): track 0.00 -> 26.2 mm
- net Net-(J5-Pad1): track 0.00 -> 13.5 mm
- net Net-(J5-Pad2): track 0.00 -> 11.3 mm
- net GPIO5: track 0.00 -> 10.7 mm
- net GPIO23: track 0.00 -> 10.7 mm
- net GPIO19: track 0.00 -> 10.7 mm
- net GPIO18: track 0.00 -> 10.7 mm
- net (no net): vias 0 -> 3
- added copper zone on B.Cu, net GND
Other:
- board outline added: 50 x 69.5 mm
- board text added: "THG v.2"

Commit message: fix cordinate
Parts:
- moved J4 33.9 mm to (155.5, 115.2), turned to 0 degrees
- moved R2 29.3 mm to (162.6, 61.1), turned to -90 degrees
- moved R1 29.0 mm to (157.5, 61.2), turned to -90 degrees
- moved S1 27.4 mm to (179.5, 85.4)
- moved J5 25.0 mm to (180.2, 104.9)
- moved R3 24.1 mm to (162.5, 83.0)
- moved PS1 23.0 mm to (171.8, 104.8)
- moved U1 22.4 mm to (160.7, 67.2)
- moved J2 20.5 mm to (141.9, 73.6)
- moved J3 20.5 mm to (141.9, 88.4)
- moved J1 16.8 mm to (181.0, 65.5)
Routing:
- net GPIO5: track 10.7 -> 59.4 mm
- net GPIO23: track 10.7 -> 56.0 mm
- net GPIO19: track 10.7 -> 52.4 mm
- net GPIO18: track 10.7 -> 48.6 mm
- net +5V: track 171.6 -> 195.7 mm
- net GND: track 156.2 -> 134.3 mm
- net Net-(S1-Pad1): track 26.2 -> 9.16 mm
- net Net-(J5-Pad1): track 13.5 -> 8.43 mm
- net SDA: track 74.8 -> 71.2 mm
- net Net-(J5-Pad2): track 11.3 -> 8.40 mm
- net SCL: track 60.7 -> 63.3 mm
- net (no net): vias 3 -> 4
- added copper zone on B.Cu, net +5V
- removed copper zone on B.Cu, net GND
Other:
- board size 50 x 69.5 mm -> 46.7 x 68.9 mm

Commit message: rev
Parts:
- J1: value AM2315_Conn -> AM2315_Jack; footprint Connector_JST:JST_EH_B4B-EH-A_1x04_P2.50mm_Vertical -> Lib_Kicad:TRRS-PJ-320A
- moved J1 16.1 mm to (180.5, 49.4), turned to 0 degrees
Routing:
- net SDA: track 71.2 -> 65.9 mm
- net +5V: track 195.7 -> 200.8 mm
- net SCL: track 63.3 -> 59.6 mm
- net (no net): vias 4 -> 3
- added copper zone on B.Cu, net GND
- removed copper zone on B.Cu, net +5V
Other:
- outline, holes or cut-outs redrawn

Commit message: revisi
Parts:
- added G***: LOGO, pic_kicad:otori_footprint, B.Cu at (143.2, 110.2)
- added G***: LOGO, pic_kicad:wifi, B.Cu at (151.6, 120.8)
- added H1: MountingHole_Pad, MountingHole:MountingHole_2.2mm_M2_Pad_Via, F.Cu at (169.6, 133.6)
- added H2: MountingHole_Pad, MountingHole:MountingHole_2.2mm_M2_Pad_Via, F.Cu at (128.8, 133.6)
- added H3: MountingHole_Pad, MountingHole:MountingHole_2.2mm_M2_Pad_Via, F.Cu at (128.8, 70.7)
- moved J2 22.6 mm to (128.7, 91.9)
- moved J3 22.6 mm to (128.7, 106.7)
- moved R1 22.6 mm to (144.3, 79.5)
- moved J1 22.6 mm to (167.3, 67.7)
- moved J4 22.6 mm to (142.3, 133.5)
- moved J5 22.6 mm to (167.1, 123.2)
- moved R3 22.6 mm to (149.4, 101.3)
- moved S1 22.6 mm to (166.4, 103.7)
- moved U1 22.6 mm to (147.5, 85.6)
- moved R2 22.6 mm to (149.4, 79.4)
- moved PS1 22.6 mm to (158.7, 123.1)
Routing:
- net (no net): vias 3 -> 0
Other:
- outline, holes or cut-outs redrawn

Commit message: Revisi 2
Parts:
- moved J4 57.0 mm to (167.8, 82.5), turned to -90 degrees
- moved G*** 17.5 mm to (134.2, 121.5)
- moved R3 9.99 mm to (141.8, 94.8)
- moved G*** 3.79 mm to (143.2, 114.0)
- moved J1 1.13 mm to (168.0, 66.8)
Routing:
- net +5V: track 200.8 -> 126.7 mm
- net GPIO5: track 59.4 -> 10.3 mm
- net GPIO23: track 56.0 -> 10.7 mm
- net GPIO19: track 52.4 -> 10.6 mm
- net GPIO18: track 48.6 -> 10.6 mm
- net GND: track 134.7 -> 105.0 mm
- net Net-(R3-Pad2): track 9.16 -> 20.4 mm
- net SCL: track 59.5 -> 65.2 mm
- net SDA: track 65.9 -> 70.7 mm

Commit message: revisi 3
Parts:
- moved J4 56.9 mm to (141.8, 133.2), turned to 0 degrees
- moved R3 6.70 mm to (141.7, 101.5)
- moved J2 4.04 mm to (127.8, 88.0)
- moved J3 4.04 mm to (127.8, 102.8)
- moved J1 1.81 mm to (167.6, 68.5)
- moved U1 0.08 mm to (147.4, 85.6)
Routing:
- net GND: track 105.0 -> 269.6 mm
- net +5V: track 126.7 -> 213.9 mm
- net GPIO5: track 10.3 -> 60.0 mm
- net GPIO23: track 10.7 -> 56.8 mm
- net GPIO19: track 10.6 -> 53.2 mm
- net GPIO18: track 10.6 -> 48.7 mm
- net Net-(R3-Pad2): track 20.4 -> 14.5 mm
- net SCL: track 65.2 -> 68.3 mm
- net SDA: track 70.7 -> 73.8 mm
Other:
- board size 46.7 x 68.9 mm -> 47.9 x 68.9 mm

Commit message: revisi tata letak dan rangkaian button
Parts:
- R3: value n/a -> 10k
- moved U1 3.54 mm to (147.5, 89.2)
Connections:
- H1 pad 1: GND -> unconnected-(H1-Pad1)
- S1 pad 2: GND -> GPIO35
- U1 pad 7: unconnected-(U1-Pad7) -> GPIO35
Routing:
- net GND: track 269.6 -> 164.6 mm
- net GPIO35: track 0.00 -> 9.70 mm
- net SDA: track 73.8 -> 79.5 mm
- net GPIO23: track 56.8 -> 51.5 mm
- net GPIO5: track 60.0 -> 54.9 mm
- net GPIO19: track 53.2 -> 48.1 mm
- net GPIO18: track 48.7 -> 44.8 mm
- net unconnected-(H1-Pad1): track 0.00 -> 2.02 mm
- net SCL: track 68.3 -> 69.9 mm
