File: PCB/MARUKO_Analog_PoC/MARUKO_Analog/MARUKO_Analog.kicad_pcb (KiCad board)
At the start: 2 copper layers, 132.1 x 115 mm, 119 parts, among them J1 Asus_Tinkerboard_sR2.0, J10 Fan 12V, J11 indicator, J2 CONMHF4-SMD-G-T, J3 Sensor 4, J4 Sensor 3, J5 Sensor 2, J6 Sensor 1, J7 Power In 24v, K1 G3MB202PDC12, Q1 2N3904, Q2 2N3904, Q3 2N3904, Q4 2N3904, Q5 BC548, Q6 BC548, SW1 Button 1, SW2 Button 2, U1 LM358, U10 LM358, U11 LM358, U12 LM358, U13 ADS1115, U14 RFM95W-915S2, U16 MP1584_Module, U17 MP1584_Module, U18 MP1584_Module, U2 LM358, U3 LM358, U4 LM358, U5 HCNR200, U6 HCNR200, U7 HCNR200, U8 HCNR200, U9 LM358

Commit message: generate gerber file of modbus rev2
Changed lines of the file:
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@@
       (outputformat 1)
       (mirror false)
-      (drillshape 1)
+      (drillshape 0)
       (scaleselection 1)
       (outputdirectory "")
@@
     (fp_line (start 4.95 -2.35) (end -2.45 -2.35) (layer "F.Fab") (width 0.1))
     (fp_line (start -2.45 -2.35) (end -2.45 3.4) (layer "F.Fab") (width 0.1))
-    (pad "1" thru_hole roundrect (at 0 0) (size 1.7 2) (drill 1) (layers *.Cu *.Mask) (roundrect_rratio 0.147059)
+    (pad "1" thru_hole roundrect (at 0 0) (size 1.7 2) (drill 1) (layers *.Cu *.Mask) (roundrect_rratio 0.1470588235)
       (net 24 "+12V") (pinfunction "Pin_1") (pintype "passive"))
     (pad "2" thru_hole oval (at 2.5 0) (size 1.7 2) (drill 1) (layers *.Cu *.Mask)
@@
     (fp_line (start -0.625 -2.35) (end 0 -1.35) (layer "F.Fab") (width 0.1))
     (fp_line (start 9.95 -2.35) (end -2.45 -2.35) (layer "F.Fab") (width 0.1))
-    (pad "1" thru_hole roundrect (at 0 0 270) (size 1.7 1.95) (drill 0.95) (layers *.Cu *.Mask) (roundrect_rratio 0.147059)
+    (pad "1" thru_hole roundrect (at 0 0 270) (size 1.7 1.95) (drill 0.95) (layers *.Cu *.Mask) (roundrect_rratio 0.1470588235)
       (net 2 "Earth") (pinfunction "Pin_1") (pintype "passive"))
     (pad "2" thru_hole oval (at 2.5 0 270) (size 1.7 1.95) (drill 0.95) (layers *.Cu *.Mask)
@@
     (fp_line (start 7.45 -2.35) (end -2.45 -2.35) (layer "F.Fab") (width 0.1))
     (fp_line (start -0.625 -2.35) (end 0 -1.35) (layer "F.Fab") (width 0.1))
-    (pad "1" thru_hole roundrect (at 0 0) (size 1.7 1.95) (drill 0.95) (layers *.Cu *.Mask) (roundrect_rratio 0.147059)
+    (pad "1" thru_hole roundrect (at 0 0) (size 1.7 1.95) (drill 0.95) (layers *.Cu *.Mask) (roundrect_rratio 0.1470588235)
       (net 64 "Input 2") (pinfunction "Pin_1") (pintype "passive"))
     (pad "2" thru_hole oval (at 2.5 0) (size 1.7 1.95) (drill 0.95) (layers *.Cu *.Mask)
@@
     (fp_line (start 7.45 3.4) (end 7.45 -2.35) (layer "F.Fab") (width 0.1))
     (fp_line (start -2.45 -2.35) (end -2.45 3.4) (layer "F.Fab") (width 0.1))
-    (pad "1" thru_hole roundrect (at 0 0) (size 1.7 1.95) (drill 0.95) (layers *.Cu *.Mask) (roundrect_rratio 0.147059)
+    (pad "1" thru_hole roundrect (at 0 0) (size 1.7 1.95) (drill 0.95) (layers *.Cu *.Mask) (roundrect_rratio 0.1470588235)
       (net 63 "Input 1") (pinfunction "Pin_1") (pintype "passive"))
     (pad "2" thru_hole oval (at 2.5 0) (size 1.7 1.95) (drill 0.95) (layers *.Cu *.Mask)
@@
     (fp_line (start -2.45 -2.35) (end -2.45 3.4) (layer "F.Fab") (width 0.1))
     (fp_line (start 7.45 -2.35) (end -2.45 -2.35) (layer "F.Fab") (width 0.1))
-    (pad "1" thru_hole roundrect (at 0 0) (size 1.7 1.95) (drill 0.95) (layers *.Cu *.Mask) (roundrect_rratio 0.147059)
+    (pad "1" thru_hole roundrect (at 0 0) (size 1.7 1.95) (drill 0.95) (layers *.Cu *.Mask) (roundrect_rratio 0.1470588235)
       (net 68 "Input 4") (pinfunction "Pin_1") (pintype "passive"))
     (pad "2" thru_hole oval (at 2.5 0) (size 1.7 1.95) (drill 0.95) (layers *.Cu *.Mask)
@@
     (fp_line (start 7.45 -2.35) (end -2.45 -2.35) (layer "F.Fab") (width 0.1))
     (fp_line (start -2.45 3.4) (end 7.45 3.4) (layer "F.Fab") (width 0.1))
-    (pad "1" thru_hole roundrect (at 0 0) (size 1.7 1.95) (drill 0.95) (layers *.Cu *.Mask) (roundrect_rratio 0.147059)
+    (pad "1" thru_hole roundrect (at 0 0) (size 1.7 1.95) (drill 0.95) (layers *.Cu *.Mask) (roundrect_rratio 0.1470588235)
       (net 66 "Input 3") (pinfunction "Pin_1") (pintype "passive"))
     (pad "2" thru_hole oval (at 2.5 0) (size 1.7 1.95) (drill 0.95) (layers *.Cu *.Mask)
