File: PCB/MARUKO_RS485_Rev2/MARUKO_RS485_Rev2.kicad_pcb (KiCad board)
At the start: 2 copper layers, 105 x 65 mm, 49 parts, among them J1 Sensor 1, J2 Sensor 2, J3 Sensor 3, J4 sensor 4, J5 Asus_Tinkerboard_sR2.0, J6 LED Indicator, J7 CONMHF4-SMD-G-T, J8 Power In 24v, J9 Fan 12V, K1 G3MB202PDC12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

Commit message: generate gerber file of modbus rev2
Parts:
- removed REF**: MODULE_RASPBERRY_PI_3_MODEL_B+, Lib_Kicad:MODULE_RASPBERRY_PI_3_MODEL_B+
Routing:
- net 24V_System: track 17.1 -> 19.7 mm
- net +5V: track 127.8 -> 130.4 mm
- net +24V: track 167.4 -> 169.9 mm
- net +12V: track 108.0 -> 110.5 mm
